File: circuits/C.H.I.P./C.H.I.P..kicad_pcb (KiCad board)
At the start: 2 copper layers, 40.6 x 55.2 mm, 40 parts, among them J13 DIP-HEADER-2x20, J14 DIP-HEADER-2x20, P0 CONN_01X03, P0-1 CONN_01X03, P1-0 CONN_01X03, P1-1 CONN_01X03, P2-0 CONN_01X02, P2-1 CONN_01X02, P3-0 CONN_01X02, P3-1 CONN_01X02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

Commit message: update the C.H.I.P. design and add the gerbers
Other:
- board text added: "IN"
- board text added: "OUT"
Changed lines of the file:
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@@
     (area 67.678 51.461999 178.510001 123.265001)
     (thickness 1.6)
-    (drawings 68)
+    (drawings 72)
     (tracks 203)
     (zones 0)
@@
   )
   (setup
-    (last_trace_width 0.1524)
+    (last_trace_width 0.254)
     (user_trace_width 0.1524)
     (user_trace_width 0.254)
@@
     )
   )
+  (gr_text IN (at 96.8375 70.104 90) (layer F.SilkS)
+    (effects (font (size 1.2 1.2) (thickness 0.3)))
+  )
+  (gr_text OUT (at 93.599 70.0405 90) (layer F.SilkS)
+    (effects (font (size 1.2 1.2) (thickness 0.3)))
+  )
+  (gr_text OUT (at 88.2015 70.0405 90) (layer F.SilkS)
+    (effects (font (size 1.2 1.2) (thickness 0.3)))
+  )
+  (gr_text IN (at 85.0265 70.104 90) (layer F.SilkS)
+    (effects (font (size 1.2 1.2) (thickness 0.3)))
+  )
   (gr_line (start 111.0615 52.197) (end 111.0615 51.6255) (angle 90) (layer F.SilkS) (width 0.2))
